Commit message: chore: 절대 경로 -> 상대경로로 수정

File: asset/doosan_e0509/e0509_with_gripper.urdf (robot description, URDF)
Before this commit: robot e0509, 13 links, 12 joints
Links:
- link base_link: geometry collision mesh filename=configurations/e0509_collision/E0509_0_0.dae scale=0.001 0.001 0.001; visual mesh filename=configurations/e0509_white/E0509_0_0.dae scale=0.001 0.001 0.001
- link link_1: geometry collision mesh filename=configurations/e0509_collision/E0509_1_1.dae scale=0.001 0.001 0.001; collision mesh filename=configurations/e0509_collision/E0509_1_2.dae scale=0.001 0.001 0.001
- link link_2: geometry collision mesh filename=configurations/e0509_collision/E0509_2_1.dae scale=0.001 0.001 0.001; collision mesh filename=configurations/e0509_collision/E0509_2_2.dae scale=0.001 0.001 0.001
- link link_3: geometry collision mesh filename=configurations/e0509_collision/E0509_3_1.dae scale=0.001 0.001 0.001; collision mesh filename=configurations/e0509_collision/E0509_3_2.dae scale=0.001 0.001 0.001
- link link_4: geometry collision mesh filename=configurations/e0509_collision/E0509_4_1.dae scale=0.001 0.001 0.001; collision mesh filename=configurations/e0509_collision/E0509_4_2.dae scale=0.001 0.001 0.001
- link link_5: geometry collision mesh filename=configurations/e0509_collision/E0509_5_1.dae scale=0.001 0.001 0.001; collision mesh filename=configurations/e0509_collision/E0509_5_2.dae scale=0.001 0.001 0.001
- link link_6: geometry collision mesh filename=configurations/e0509_collision/E0509_6_1.dae scale=0.001 0.001 0.001; visual mesh filename=configurations/e0509_white/E0509_6_1.dae scale=0.001 0.001 0.001
- link rh_p12_rn_base: geometry collision mesh filename=configurations/e0509_collision/base.stl scale=0.001 0.001 0.001; visual mesh filename=configurations/e0509_collision/base.stl scale=0.001 0.001 0.001
- link rh_p12_rn_l1: geometry collision mesh filename=configurations/e0509_collision/l1.stl scale=0.001 0.001 0.001; visual mesh filename=configurations/e0509_collision/l1.stl scale=0.001 0.001 0.001
- link rh_p12_rn_l2: geometry collision mesh filename=configurations/e0509_collision/l2.stl scale=0.001 0.001 0.001; visual mesh filename=configurations/e0509_collision/l2.stl scale=0.001 0.001 0.001
- link rh_p12_rn_r1: geometry collision mesh filename=configurations/e0509_collision/r1.stl scale=0.001 0.001 0.001; visual mesh filename=configurations/e0509_collision/r1.stl scale=0.001 0.001 0.001
- link rh_p12_rn_r2: geometry collision mesh filename=configurations/e0509_collision/r2.stl scale=0.001 0.001 0.001; visual mesh filename=configurations/e0509_collision/r2.stl scale=0.001 0.001 0.001
